File: supply/supply.sch (EAGLE design)
At the start: 14 parts, among them IC3 R-78E3.3-0.5, J1 DIN5, J2 1X2-3.5MM

Commit message: Redo supply to be much simpler
Parts:
- removed C10: 10u, rcl:CPOL-USA
- removed C19, C20: 22u, rcl:C-USC1206
- removed C24, C26: 22u, rcl:CPOL-USB
- removed C7: 100n, rcl:C-USC0402
- removed D1, D2: 1N4001, gm-diodes:1N400X.3
- removed IC3: R-78E3.3-0.5, og-vreg:WE173950378
- removed L1: 33u, og-rcl:L-USL2012C
- J2: value 1X2-3.5MM -> (none); device adafruit:1X2-3.5MM -> SparkFun-Connectors:CONN_02
Connections:
- removed net +3V3: C10.+, C7.1, IC3.VO, J2.1
- removed net N$1: C19.1, IC3.VI, L1.2
- removed net N$2: D1.A, J1.3
- removed net N$3: D2.C, J1.1
- new net +5V: J1.3, J2.1
- net GND: now also J1.1, JP2.1, JP2.3, JP2.5, JP2.7, JP2.9; no longer C10.-, C19.2, C20.2, C24.-, C26.+, C7.2, IC3.GND, JP2.10, JP2.2, JP2.4, JP2.6, JP2.8
- net VCC: now also J1.5; no longer C20.1, C24.+, D1.C, L1.1
- net VEE: now also J1.4, JP2.10, JP2.2, JP2.4, JP2.6, JP2.8; no longer C26.-, D2.A, JP2.1, JP2.3, JP2.5, JP2.7, JP2.9
Other:
- note added: "TODO: double check pinout, make sure header is correct"
- note removed: "Need to pinout DIN5 connector"
